Commit message: aaaaaaaaaaaaa

File: test_urdf.urdf (robot description, URDF)
Before this commit: robot axaxabot, 6 links, 5 joints
Links:
- link robot_base: geometry collision mesh filename=package://src/abot_description/meshes/robot_base.stl; visual mesh filename=package://src/abot_description/meshes/robot_base.stl
- link robot_caster_wheel_1: geometry collision mesh filename=package://src/abot_description/meshes/robot_wheel_r.stl; visual mesh filename=package://src/abot_description/meshes/robot_wheel_center.stl
- link robot_caster_wheel_2: geometry collision mesh filename=package://src/abot_description/meshes/robot_wheel_r.stl; visual mesh filename=package://src/abot_description/meshes/robot_wheel_center.stl
- link robot_left_wheel: geometry collision mesh filename=package://src/abot_description/meshes/robot_wheel_l.stl; visual mesh filename=package://src/abot_description/meshes/robot_wheel_l.stl
- link robot_right_wheel: geometry collision mesh filename=package://src/abot_description/meshes/robot_wheel_r.stl; visual mesh filename=package://src/abot_description/meshes/robot_wheel_r.stl

Commit message: remaked path

File: test_urdf.urdf (robot description, URDF)
Before this commit: robot axaxabot, 6 links, 5 joints
Links:
- link robot_base: geometry collision mesh filename=/home/ubuntu/ros/src/abot_description/meshes/robot_base.stl; visual mesh filename=/home/ubuntu/ros/src/abot_description/meshes/robot_base.stl
- link robot_caster_wheel_1: geometry collision mesh filename=/home/ubuntu/ros/src/abot_description/meshes/robot_wheel_r.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; visual mesh filename=/home/ubuntu/ros/src/abot_description/meshes/robot_wheel_ce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
- link robot_caster_wheel_2: geometry collision mesh filename=/home/ubuntu/ros/src/abot_description/meshes/robot_wheel_r.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; visual mesh filename=/home/ubuntu/ros/src/abot_description/meshes/robot_wheel_ce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
- link robot_left_wheel: geometry collision mesh filename=/home/ubuntu/ros/src/abot_description/meshes/robot_wheel_l.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; visual mesh filename=/home/ubuntu/ros/src/abot_description/meshes/robot_wheel_l.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
- link robot_right_wheel: geometry collision mesh filename=/home/ubuntu/ros/src/abot_description/meshes/robot_wheel_r.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; visual mesh filename=/home/ubuntu/ros/src/abot_description/meshes/robot_wheel_r.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
