Commit message: new files

File: urdf/urdf_v1.urdf (robot description, URDF)
Before this commit: robot axaxabot, 6 links, 5 joints
Links:
- link robot_base: geometry collision mesh filename=package://robot_description/meshes/robot_base.stl; visual mesh filename=package://robot_description/meshes/robot_base.stl
- link robot_caster_wheel_1: geometry collision mesh filename=package://robot_description/meshes/robot_wheel_r.stl; visual mesh filename=package://robot_description/meshes/robot_wheel_center.stl
- link robot_caster_wheel_2: geometry collision mesh filename=package://robot_description/meshes/robot_wheel_r.stl; visual mesh filename=package://robot_description/meshes/robot_wheel_center.stl
- link robot_left_wheel: geometry collision mesh filename=package://robot_description/meshes/robot_wheel_l.stl; visual mesh filename=package://robot_description/meshes/robot_wheel_l.stl
- link robot_right_wheel: geometry collision mesh filename=package://robot_description/meshes/robot_wheel_r.stl; visual mesh filename=package://robot_description/meshes/robot_wheel_r.stl
