Commit message: changed color

File: abot_description/urdf/abot_caster_wheel.xacro (robot description, xacro)
@@ -13,5 +13,5 @@
 				<mesh filename="package://abot_description/meshes/abot_caster_wheel.STL" />
 			</geometry>
-			<material name="Red" />
+			<material name="Green" />
 		</visual>
 		<collision>
@@ -33,5 +33,5 @@
 				<mesh filename="package://abot_description/meshes/abot_caster_wheel.STL" />
 			</geometry>
-			<material name="Red" />
+			<material name="Green" />
 		</visual>
 		<collision>
