Commit message: fixed urdf

File: abot_description/urdf/abot.xacro (robot description, xacro)
@@ -27,5 +27,5 @@
 	<link name="abot_base">
 		<inertial>
-			<origin xyz="-0.017258 -0.00044491 0.079113" rpy="0 0 0"/>
+			<origin xyz="0 0 0.0075" rpy="0 0 0"/>
 			<mass value="0.71798"/>
 			<inertia ixx="0.00077488" ixy="-3.248E-06" ixz="-9.2329E-06" iyy="0.00075836" iyz="2.2456E-06" izz="0.0014158"/>

Commit message: rename

File: abot_description/urdf/abot.xacro (robot description, xacro)
@@ -25,5 +25,5 @@
 		</visual>
 	</link>
-	<link name="abot_base">
+	<link name="robot_base">
 		<inertial>
 			<origin xyz="0 0 0.0075" rpy="0 0 0"/>
@@ -48,5 +48,5 @@
 		<origin xyz="0 0 0" rpy="0 0 0" />
 		<parent link="base_link" />
-		<child link="abot_base" />
+		<child link="robot_base" />
 	</joint>
 	<joint name="base_footprint_to_base_link" type="fixed">

File: abot_description/urdf/abot_caster_wheel.xacro (robot description, xacro)
@@ -2,5 +2,5 @@
 <robot name="abot"
 	xmlns:xacro="http://www.ros.org/wiki/xacro">
-	<link name="abot_caster_wheel_1">
+	<link name="robot_caster_wheel_1">
 		<inertial>
 			<origin xyz="0 1.6073E-19 0" rpy="0 0 0"/>
@@ -22,5 +22,5 @@
 		</collision>
 	</link>
-	<link name="abot_caster_wheel_2">
+	<link name="robot_caster_wheel_2">
 		<inertial>
 			<origin xyz="0 1.6073E-19 0" rpy="0 0 0"/>
@@ -44,12 +44,12 @@
 	<joint name="caster_wheel_1_to_base" type="continuous">
 		<origin xyz="-0.065 0 0.0075" rpy="0 0 0" />
-		<parent link="abot_base" />
-		<child link="abot_caster_wheel_1" />
+		<parent link="robot_base" />
+		<child link="robot_caster_wheel_1" />
 		<axis xyz="0 1 0" />
 	</joint>
 	<joint name="caster_wheel_2_to_base" type="continuous">
 		<origin xyz="0.055 0 0.0075" rpy="0 0 0" />
-		<parent link="abot_base" />
-		<child link="abot_caster_wheel_2" />
+		<parent link="robot_base" />
+		<child link="robot_caster_wheel_2" />
 		<axis xyz="0 1 0" />
 	</joint>

File: abot_description/urdf/abot_left_wheel.xacro (robot description, xacro)
@@ -2,5 +2,5 @@
 <robot name="abot"
 	xmlns:xacro="http://www.ros.org/wiki/xacro">
-	<link name="abot_left_wheel">
+	<link name="robot_left_wheel">
 		<inertial>
 			<origin xyz="1.9255E-10 0.00056576 -1.0414E-10" rpy="0 0 0"/>
@@ -37,12 +37,12 @@
 		</collision>
 	</link>
-	<joint name="left_wheel_to_abot_left_wheel" type="fixed">
+	<joint name="left_wheel_to_rbot_left_wheel" type="fixed">
 		<origin xyz="0 0 0" rpy="0 0 0" />
 		<parent link="left_wheel" />
-		<child link="abot_left_wheel" />
+		<child link="robot_left_wheel" />
 	</joint>
 	<joint name="left_wheel_to_base" type="continuous">
 		<origin xyz="0 -0.0896 0.0344" rpy="0 0 0" />
-		<parent link="abot_base" />
+		<parent link="robot_base" />
 		<child link="left_wheel" />
 		<axis xyz="0 1 0" />

File: abot_description/urdf/abot_right_wheel.xacro (robot description, xacro)
@@ -2,5 +2,5 @@
 <robot name="abot"
 	xmlns:xacro="http://www.ros.org/wiki/xacro">
-	<link name="abot_right_wheel">
+	<link name="robot_right_wheel">
 		<inertial>
 			<origin xyz="1.9255E-10 -0.00056576 1.0414E-10" rpy="0 0 0"/>
@@ -37,12 +37,12 @@
 		</collision>
 	</link>
-	<joint name="right_wheel_to_abot_right_wheel" type="fixed">
+	<joint name="right_wheel_to_robot_right_wheel" type="fixed">
 		<origin xyz="0 0 0" rpy="0 0 0" />
 		<parent link="right_wheel" />
-		<child link="abot_right_wheel" />
+		<child link="robot_right_wheel" />
 	</joint>
 	<joint name="right_wheel_to_base" type="continuous">
 		<origin xyz="0 0.0896 0.0344" rpy="0 0 0" />
-		<parent link="abot_base" />
+		<parent link="robot_base" />
 		<child link="right_wheel" />
 		<axis xyz="0 1 0" />

File: abot_description/urdf/abot_sensors.xacro (robot description, xacro)
@@ -2,5 +2,5 @@
 <robot name="abot"
 	xmlns:xacro="http://www.ros.org/wiki/xacro">
-	<link name="abot_lidar">
+	<link name="robot_lidar">
 		<inertial>
 			<origin xyz="0 0 0" rpy="0 0 0"/>
@@ -24,6 +24,6 @@
 	<joint name="lidar_to_base" type="fixed">
 		<origin xyz="-0.06 0.0002 0.15" rpy="0 0 ${PI}"/>
-		<parent link="abot_base"/>
-		<child link="abot_lidar"/>
+		<parent link="robot_base"/>
+		<child link="robot_lidar"/>
 		<axis xyz="0 0 0"/>
 	</joint>

Commit message: down

File: abot_description/urdf/abot.xacro (robot description, xacro)
@@ -2,5 +2,5 @@
 <robot name="abot"
 	xmlns:xacro="http://www.ros.org/wiki/xacro">
-	<xacro:property name="clearance" value="0.018" />
+	<xacro:property name="clearance" value="0.0075" />
 	<xacro:property name="wheel_radius" value="0.03195"/>
 	<xacro:property name="wheel_separation" value="0.128"/>
@@ -20,5 +20,5 @@
 			<origin xyz="0 0 0" rpy="0 0 0" />
 			<geometry>
-				<cylinder length="0.001" radius="0.100" />
+				<cylinder length="0.001" radius="0.150" />
 			</geometry>
 			<material name="Blue" />
@@ -27,5 +27,5 @@
 	<link name="robot_base">
 		<inertial>
-			<origin xyz="0 0 0.0075" rpy="0 0 0"/>
+			<origin xyz="-0.017258 -0.00044491 0.079113" rpy="0 0 0"/>
 			<mass value="0.71798"/>
 			<inertia ixx="0.00077488" ixy="-3.248E-06" ixz="-9.2329E-06" iyy="0.00075836" iyz="2.2456E-06" izz="0.0014158"/>

Commit message: and down and down

File: abot_description/urdf/abot.xacro (robot description, xacro)
@@ -2,5 +2,5 @@
 <robot name="abot"
 	xmlns:xacro="http://www.ros.org/wiki/xacro">
-	<xacro:property name="clearance" value="0.0075" />
+	<xacro:property name="clearance" value="0" />
 	<xacro:property name="wheel_radius" value="0.03195"/>
 	<xacro:property name="wheel_separation" value="0.128"/>

Commit message: radius was changed

File: abot_description/urdf/abot.xacro (robot description, xacro)
@@ -3,5 +3,5 @@
 	xmlns:xacro="http://www.ros.org/wiki/xacro">
 	<xacro:property name="clearance" value="0" />
-	<xacro:property name="wheel_radius" value="0.03195"/>
+	<xacro:property name="wheel_radius" value="0.0344"/>
 	<xacro:property name="wheel_separation" value="0.128"/>
 	<xacro:property name="wheel_width" value="0.026"/>

Commit message: new packages

File: abot_description/urdf/abot.xacro (robot description, xacro)
@@ -4,5 +4,5 @@
 	<xacro:property name="clearance" value="0" />
 	<xacro:property name="wheel_radius" value="0.0344"/>
-	<xacro:property name="wheel_separation" value="0.128"/>
+	<xacro:property name="wheel_separation" value="0.152"/>
 	<xacro:property name="wheel_width" value="0.026"/>
 	<xacro:property name="PI" value="3.1415926"/>

Commit message: new settings

File: abot_description/urdf/abot.xacro (robot description, xacro)
@@ -3,5 +3,5 @@
 	xmlns:xacro="http://www.ros.org/wiki/xacro">
 	<xacro:property name="clearance" value="0" />
-	<xacro:property name="wheel_radius" value="0.0344"/>
+	<xacro:property name="wheel_radius" value="0.1"/>
 	<xacro:property name="wheel_separation" value="0.152"/>
 	<xacro:property name="wheel_width" value="0.026"/>
@@ -20,5 +20,5 @@
 			<origin xyz="0 0 0" rpy="0 0 0" />
 			<geometry>
-				<cylinder length="0.001" radius="0.150" />
+				<cylinder length="0.001" radius="0.250" />
 			</geometry>
 			<material name="Blue" />
@@ -26,9 +26,4 @@
 	</link>
 	<link name="robot_base">
-		<inertial>
-			<origin xyz="-0.017258 -0.00044491 0.079113" rpy="0 0 0"/>
-			<mass value="0.71798"/>
-			<inertia ixx="0.00077488" ixy="-3.248E-06" ixz="-9.2329E-06" iyy="0.00075836" iyz="2.2456E-06" izz="0.0014158"/>
-		</inertial>
 		<visual>
 			<origin xyz="0 0 0" rpy="0 0 0" />
@@ -46,5 +41,5 @@
 	</link>
 	<joint name="base_link_to_abot_base" type="fixed">
-		<origin xyz="0 0 0" rpy="0 0 0" />
+		<origin xyz="0 0 0.02" rpy="0 0 0" />
 		<parent link="base_link" />
 		<child link="robot_base" />

File: abot_description/urdf/abot_caster_wheel.xacro (robot description, xacro)
@@ -3,9 +3,4 @@
 	xmlns:xacro="http://www.ros.org/wiki/xacro">
 	<link name="robot_caster_wheel_1">
-		<inertial>
-			<origin xyz="0 1.6073E-19 0" rpy="0 0 0"/>
-			<mass value="0.011207"/>
-			<inertia ixx="2.1965E-07" ixy="-1.5533E-55" ixz="-1.9776E-56" iyy="2.1965E-07" iyz="-2.2674E-40" izz="2.1965E-07"/>
-		</inertial>
 		<visual>
 			<origin xyz="0 0 0" rpy="0 0 0" />
@@ -13,5 +8,5 @@
 				<mesh filename="package://abot_description/meshes/abot_caster_wheel.STL" />
 			</geometry>
-			<material name="Green" />
+			<material name="Red" />
 		</visual>
 		<collision>
@@ -23,9 +18,4 @@
 	</link>
 	<link name="robot_caster_wheel_2">
-		<inertial>
-			<origin xyz="0 1.6073E-19 0" rpy="0 0 0"/>
-			<mass value="0.011207"/>
-			<inertia ixx="2.1965E-07" ixy="-1.5533E-55" ixz="-1.9776E-56" iyy="2.1965E-07" iyz="-2.2674E-40" izz="2.1965E-07"/>
-		</inertial>
 		<visual>
 			<origin xyz="0 0 0" rpy="0 0 0" />
@@ -33,5 +23,5 @@
 				<mesh filename="package://abot_description/meshes/abot_caster_wheel.STL" />
 			</geometry>
-			<material name="Green" />
+			<material name="Red" />
 		</visual>
 		<collision>
@@ -43,5 +33,5 @@
 	</link>
 	<joint name="caster_wheel_1_to_base" type="continuous">
-		<origin xyz="-0.065 0 0.0075" rpy="0 0 0" />
+		<origin xyz="-0.13 0 -0.015" rpy="0 0 0" />
 		<parent link="robot_base" />
 		<child link="robot_caster_wheel_1" />
@@ -49,5 +39,5 @@
 	</joint>
 	<joint name="caster_wheel_2_to_base" type="continuous">
-		<origin xyz="0.055 0 0.0075" rpy="0 0 0" />
+		<origin xyz="0.13 0 -0.015" rpy="0 0 0" />
 		<parent link="robot_base" />
 		<child link="robot_caster_wheel_2" />

File: abot_description/urdf/abot_left_wheel.xacro (robot description, xacro)
@@ -3,9 +3,4 @@
 	xmlns:xacro="http://www.ros.org/wiki/xacro">
 	<link name="robot_left_wheel">
-		<inertial>
-			<origin xyz="1.9255E-10 0.00056576 -1.0414E-10" rpy="0 0 0"/>
-			<mass value="0.050464"/>
-			<inertia ixx="2.0701E-05" ixy="-3.8089E-14" ixz="1.3584E-15" iyy="3.5827E-05" iyz="2.1838E-15" izz="2.0701E-05"/>
-		</inertial>
 		<visual>
 			<origin xyz="0 0 0" rpy="0 0 0" />
@@ -13,5 +8,5 @@
 				<mesh filename="package://abot_description/meshes/abot_left_wheel.STL" />
 			</geometry>
-			<material name="Green" />
+			<material name="Red" />
 		</visual>
 		<collision>
@@ -28,5 +23,5 @@
 				<cylinder length="${wheel_width}" radius="${wheel_radius}"/>
 			</geometry>
-			<material name="Green" />
+			<material name="Red" />
 		</visual>
 		<collision>
@@ -37,5 +32,5 @@
 		</collision>
 	</link>
-	<joint name="left_wheel_to_rbot_left_wheel" type="fixed">
+	<joint name="left_wheel_to_robot_left_wheel" type="fixed">
 		<origin xyz="0 0 0" rpy="0 0 0" />
 		<parent link="left_wheel" />
@@ -43,5 +38,5 @@
 	</joint>
 	<joint name="left_wheel_to_base" type="continuous">
-		<origin xyz="0 -0.0896 0.0344" rpy="0 0 0" />
+		<origin xyz="0 0.205 0.03" rpy="0 0 0" />
 		<parent link="robot_base" />
 		<child link="left_wheel" />

File: abot_description/urdf/abot_right_wheel.xacro (robot description, xacro)
@@ -3,9 +3,4 @@
 	xmlns:xacro="http://www.ros.org/wiki/xacro">
 	<link name="robot_right_wheel">
-		<inertial>
-			<origin xyz="1.9255E-10 -0.00056576 1.0414E-10" rpy="0 0 0"/>
-			<mass value="0.050464"/>
-			<inertia ixx="2.0701E-05" ixy="3.8089E-14" ixz="-1.3584E-15" iyy="3.5827E-05" iyz="2.1838E-15" izz="2.0701E-05"/>
-		</inertial>
 		<visual>
 			<origin xyz="0 0 0" rpy="0 0 0" />
@@ -13,5 +8,5 @@
 				<mesh filename="package://abot_description/meshes/abot_right_wheel.STL" />
 			</geometry>
-			<material name="Green" />
+			<material name="Red" />
 		</visual>
 		<collision>
@@ -28,5 +23,5 @@
 				<cylinder length="${wheel_width}" radius="${wheel_radius}"/>
 			</geometry>
-			<material name="Green" />
+			<material name="Red" />
 		</visual>
 		<collision>
@@ -43,5 +38,5 @@
 	</joint>
 	<joint name="right_wheel_to_base" type="continuous">
-		<origin xyz="0 0.0896 0.0344" rpy="0 0 0" />
+		<origin xyz="0 -0.205 0.03" rpy="0 0 0" />
 		<parent link="robot_base" />
 		<child link="right_wheel" />

File: abot_description/urdf/abot_sensors.xacro (robot description, xacro)
@@ -3,9 +3,4 @@
 	xmlns:xacro="http://www.ros.org/wiki/xacro">
 	<link name="robot_lidar">
-		<inertial>
-			<origin xyz="0 0 0" rpy="0 0 0"/>
-			<mass value="0"/>
-			<inertia ixx="0" ixy="0" ixz="0" iyy="0" iyz="0" izz="0"/>
-		</inertial>
 		<visual>
 			<origin xyz="0 0 0" rpy="0 0 0"/>
@@ -23,5 +18,5 @@
 	</link>
 	<joint name="lidar_to_base" type="fixed">
-		<origin xyz="-0.06 0.0002 0.15" rpy="0 0 ${PI}"/>
+		<origin xyz="0 0 0.12" rpy="0 0 ${PI}"/>
 		<parent link="robot_base"/>
 		<child link="robot_lidar"/>

Commit message: q

File: abot_description/urdf/abot.xacro (robot description, xacro)
@@ -3,5 +3,5 @@
 	xmlns:xacro="http://www.ros.org/wiki/xacro">
 	<xacro:property name="clearance" value="0" />
-	<xacro:property name="wheel_radius" value="0.1"/>
+	<xacro:property name="wheel_radius" value="0.05"/>
 	<xacro:property name="wheel_separation" value="0.152"/>
 	<xacro:property name="wheel_width" value="0.026"/>
